File: board/WritingRobotV2.kicad_pcb (KiCad board)
At the start: 2 copper layers, 70 x 75 mm, 25 parts, among them J1 PowerSwitch, J10 DEBUG_5V, J2 MOTOR-1-OUTPUT, J3 MOTOR-2-OUTPUT, J4 CAN-INPUT, J5 POWER_INPUT, J6 Conn_01x02_Pin, J7 Conn_01x02_Pin, J8 DEBUG_GND, J9 DEBUG_12V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

Commit message: Adding everything
Parts:
- moved H3 14.9 mm to (25.0, 175.0)
- turned R2 to -90 degrees
Routing:
- net Net-(J4-Pin_1): track 18.1 -> 25.2 mm
- net Net-(J4-Pin_2): track 23.5 -> 29.1 mm
Other:
- board size 70 x 75 mm -> 94.2 x 80.3 mm
Changed lines of the file:
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@@
 	(footprint "Resistor_THT:R_Axial_DIN0204_L3.6mm_D1.6mm_P7.62mm_Horizontal"
 		(layer "F.Cu")
-		(at 90.19 166)
+		(at 90.19 166 -90)
 		(descr "Resistor, Axial_DIN0204 series, Axial, Horizontal, pin pitch=7.62mm, 0.167W, length*diameter=3.6*1.6mm^2, http://cdn-reichelt.de/documents/datenblatt/B400/1_4W%23YAG.pdf")
 		(tags "Resistor Axial_DIN0204 series Axial Horizontal pin pitch 7.62mm 0.167W length 3.6mm diameter 1.6mm")
 		(property "Reference" "R2"
-			(at 3.81 0 0)
+			(at 3.81 0 90)
 			(layer "F.SilkS")
 			(effects
@@
 		)
 		(property "Value" "60"
-			(at 18.31 0 0)
+			(at 18.31 0 90)
 			(layer "F.Fab")
 			(effects
@@
 		)
 		(property "Footprint" "Resistor_THT:R_Axial_DIN0204_L3.6mm_D1.6mm_P7.62mm_Horizontal"
-			(at 0 0 0)
+			(at 0 0 -90)
 			(unlocked yes)
 			(layer "F.Fab")
@@
 		)
 		(property "Datasheet" ""
-			(at 0 0 0)
+			(at 0 0 -90)
 			(unlocked yes)
 			(layer "F.Fab")
@@
 		)
 		(property "Description" "Resistor"
-			(at 0 0 0)
+			(at 0 0 -90)
 			(unlocked yes)
 			(layer "F.Fab")
@@
 		(attr through_hole)
 		(fp_line
-			(start 0.94 0)
-			(end 1.89 0)
+			(start 1.89 0.92)
+			(end 5.73 0.92)
 			(stroke
 				(width 0.12)
@@
 		)
 		(fp_line
-			(start 1.89 -0.92)
-			(end 1.89 0.92)
+			(start 5.73 0.92)
+			(end 5.73 -0.92)
 			(stroke
 				(width 0.12)
@@
 		)
 		(fp_line
-			(start 1.89 0.92)
-			(end 5.73 0.92)
+			(start 0.94 0)
+			(end 1.89 0)
 			(stroke
 				(width 0.12)
@@
 		)
 		(fp_line
-			(start 5.73 -0.92)
-			(end 1.89 -0.92)
+			(start 6.68 0)
+			(end 5.73 0)
 			(stroke
 				(width 0.12)
@@
 		)
 		(fp_line
-			(start 5.73 0.92)
-			(end 5.73 -0.92)
+			(start 1.89 -0.92)
+			(end 1.89 0.92)
 			(stroke
 				(width 0.12)
@@
 		)
 		(fp_line
-			(start 6.68 0)
-			(end 5.73 0)
+			(start 5.73 -0.92)
+			(end 1.89 -0.92)
 			(stroke
 				(width 0.12)
@@
 		)
 		(fp_line
-			(start -0.95 -1.05)
-			(end -0.95 1.05)
+			(start -0.95 1.05)
+			(end 8.57 1.05)
 			(stroke
 				(width 0.05)
@@
 		)
 		(fp_line
-			(start -0.95 1.05)
-			(end 8.57 1.05)
+			(start 8.57 1.05)
+			(end 8.57 -1.05)
 			(stroke
 				(width 0.05)
@@
 		)
 		(fp_line
-			(start 8.57 -1.05)
-			(end -0.95 -1.05)
+			(start -0.95 -1.05)
+			(end -0.95 1.05)
 			(stroke
 				(width 0.05)
@@
 		)
 		(fp_line
-			(start 8.57 1.05)
-			(end 8.57 -1.05)
+			(start 8.57 -1.05)
+			(end -0.95 -1.05)
 			(stroke
 				(width 0.05)
@@
 		)
 		(fp_line
-			(start 0 0)
-			(end 2.01 0)
+			(start 2.01 0.8)
+			(end 5.61 0.8)
 			(stroke
 				(width 0.1)
@@
 		)
 		(fp_line
-			(start 2.01 -0.8)
-			(end 2.01 0.8)
+			(start 5.61 0.8)
+			(end 5.61 -0.8)
 			(stroke
 				(width 0.1)
@@
 		)
 		(fp_line
-			(start 2.01 0.8)
-			(end 5.61 0.8)
+			(start 0 0)
+			(end 2.01 0)
 			(stroke
 				(width 0.1)
@@
 		)
 		(fp_line
-			(start 5.61 -0.8)
-			(end 2.01 -0.8)
+			(start 7.62 0)
+			(end 5.61 0)
 			(stroke
 				(width 0.1)
@@
 		)
 		(fp_line
-			(start 5.61 0.8)
-			(end 5.61 -0.8)
+			(start 2.01 -0.8)
+			(end 2.01 0.8)
 			(stroke
 				(width 0.1)
@@
 		)
 		(fp_line
-			(start 7.62 0)
-			(end 5.61 0)
+			(start 5.61 -0.8)
+			(end 2.01 -0.8)
 			(stroke
 				(width 0.1)
@@
 		)
 		(fp_text user "${REFERENCE}"
-			(at 18.31 -1 0)
+			(at 18.31 -1 90)
 			(layer "F.Fab")
 			(effects
@@
 		)
 		(pad "1" thru_hole circle
-			(at 0 0)
+			(at 0 0 270)
 			(size 1.4 1.4)
 			(drill 0.7)
@@
 		)
 		(pad "2" thru_hole oval
-			(at 7.62 0)
+			(at 7.62 0 270)
 			(size 1.4 1.4)
 			(drill 0.7)
@@
 	(footprint "MountingHole:MountingHole_4.3mm_M4"
 		(layer "F.Cu")
-		(at 39 180)
+		(at 25 175)
 		(descr "Mounting Hole 4.3mm, no annular, M4")
 		(tags "mounting hole 4.3mm no annular m4")
@@
 		(layer "F.SilkS")
 	)
-	(gr_rect
-		(start 35 110)
-		(end 105 185)
+	(gr_line
+		(start 104.5 107)
+		(end 108.253776 177.087303)
+		(stroke
+			(width 0.05)
+			(type default)
+		)
+		(layer "Edge.Cuts")
+	)
+	(gr_arc
+		(start 25 186.5)
+		(mid 17.618942 183.655978)
+		(end 14.054591 176.594541)
+		(stroke
+			(width 0.05)
+			(type default)
+		)
+		(layer "Edge.Cuts")
+	)
+	(gr_line
+		(start 14.054591 176.594541)
+		(end 15.5 111.5)
+		(stroke
+			(width 0.05)
+			(type default)
+		)
+		(layer "Edge.Cuts")
+	)
+	(gr_line
+		(start 63.5 106.5)
+		(end 104.5 107)
+		(stroke
+			(width 0.05)
+			(type default)
+		)
+		(layer "Edge.Cuts")
+	)
+	(gr_circle
+		(center 40.5 116)
+		(end 35 116)
 		(stroke
 			(width 0.05)
@@
 		(layer "Edge.Cuts")
 	)
+	(gr_line
+		(start 25 186.5)
+		(end 98.497329 186.758534)
+		(stroke
+			(width 0.05)
+			(type default)
+		)
+		(layer "Edge.Cuts")
+	)
+	(gr_line
+		(start 15.5 111.5)
+		(end 63.5 106.5)
+		(stroke
+			(width 0.05)
+			(type default)
+		)
+		(layer "Edge.Cuts")
+	)
+	(gr_arc
+		(start 108.253776 177.087303)
+		(mid 105.230473 183.794183)
+		(end 98.497329 186.758534)
+		(stroke
+			(width 0.05)
+			(type default)
+		)
+		(layer "Edge.Cuts")
+	)
 	(gr_text "WTF it's alive?"
 		(at 96 168.5 0)
@@
 		(layer "F.Fab")
 		(pts
-			(xy 103.5 185) (xy 103.5 110)
-		)
-		(height 25)
-		(orientation 1)
-		(gr_text "75,0000 mm"
-			(at 127.35 147.5 90)
-			(layer "F.Fab")
-			(effects
-				(font
-					(size 1 1)
-					(thickness 0.15)
-				)
-			)
-		)
-		(format
-			(prefix "")
-			(suffix "")
-			(units 3)
-			(units_format 1)
-			(precision 4)
-		)
-		(style
-			(thickness 0.1)
-			(arrow_length 1.27)
-			(text_position_mode 0)
-			(extension_height 0.58642)
-			(extension_offset 0.5) keep_text_aligned)
-	)
-	(dimension
-		(type orthogonal)
-		(layer "F.Fab")
-		(pts
 			(xy 91.5 180) (xy 39 180)
 		)
@@
 	)
 	(segment
-		(start 97.81 162.37)
-		(end 95.26 159.82)
+		(start 100.530711 174.75)
+		(end 98.500711 172.72)
+		(width 0.5)
+		(layer "F.Cu")
+		(net 48)
+	)
+	(segment
+		(start 98.500711 172.72)
+		(end 96 172.72)
 		(width 0.5)
 		(layer "F.Cu")
@@
 	)
 	(segment
-		(start 103 168.19)
+		(start 94.4 163)
 		(end 97.81 163)
 		(width 0.5)
@@
 	)
 	(segment
-		(start 97.81 163)
-		(end 97.81 162.37)
+		(start 94.4 163)
+		(end 94.4 160.68)
+		(width 0.5)
+		(layer "F.Cu")
+		(net 48)
+	)
+	(segment
+		(start 96 172.72)
+		(end 94.4 171.12)
+		(width 0.5)
+		(layer "F.Cu")
+		(net 48)
+	)
+	(segment
+		(start 94.4 171.12)
+		(end 94.4 163)
+		(width 0.5)
+		(layer "F.Cu")
+		(net 48)
+	)
+	(segment
+		(start 94.4 160.68)
+		(end 95.26 159.82)
 		(width 0.5)
 		(layer "F.Cu")
@@
 	(segment
 		(start 103 174.75)
-		(end 103 168.19)
+		(end 100.530711 174.75)
 		(width 0.5)
 		(layer "F.Cu")
@@
 	)
 	(segment
-		(start 97.81 173.302081)
-		(end 101.797919 177.29)
+		(start 95 173.62)
+		(end 98.127919 173.62)
 		(width 0.5)
 		(layer "F.Cu")
@@
 	)
 	(segment
-		(start 97.81 166)
-		(end 97.81 173.302081)
+		(start 93.5 160.6)
+		(end 92.72 159.82)
 		(width 0.5)
 		(layer "F.Cu")
@@
 	)
 	(segment
-		(start 96 166)
-		(end 92.72 162.72)
+		(start 95 173.62)
+		(end 95 173)
 		(width 0.5)
 		(layer "F.Cu")
@@
 	)
 	(segment
-		(start 101.797919 177.29)
-		(end 103 177.29)
+		(start 98.127919 173.62)
+		(end 101.797919 177.29)
 		(width 0.5)
 		(layer "F.Cu")
@@
 	)
 	(segment
-		(start 92.72 162.72)
-		(end 92.72 159.82)
+		(start 93.5 171.5)
+		(end 93.5 160.6)
+		(width 0.5)
+		(layer "F.Cu")
+		(net 49)
+	)
+	(segment
+		(start 90.19 173.62)
+		(end 95 173.62)
+		(width 0.5)
+		(layer "F.Cu")
+		(net 49)
+	)
+	(segment
+		(start 101.797919 177.29)
+		(end 103 177.29)
 		(width 0.5)
 		(layer "F.Cu")
@@
 	)
 	(segment
-		(start 97.81 166)
-		(end 96 166)
+		(start 95 173)
+		(end 93.5 171.5)
 		(width 0.5)
 		(layer "F.Cu")
